File: hardware/master/master.kicad_pcb (KiCad board)
At the start: 2 copper layers, 200 x 200 mm, 33 parts, among them U1 ATtiny1604-SS, U2 esp32-wemos-d1-mini, U3 LOGIC_LEVEL_2CH_3V3_5V

Commit message: feat: add hardware firmware suite and update KiCad master/slave PCB designs
Parts:
- moved C_LV1 21.0 mm to (136.6, 432.0)
- moved C_HV1 18.0 mm to (139.8, 416.1)
- moved R_LED1 1.50 mm to (169.0, 414.0), turned to 0 degrees
- moved C_ATTINY1 0.71 mm to (162.0, 422.5)
Routing:
- net +12V_BUS: track 0.00 -> 463.2 mm, vias 0 -> 4
- net +5V_LOCAL: track 0.00 -> 400.2 mm, vias 0 -> 5
- net LED_R3_TO_R4: track 0.00 -> 194.5 mm
- net LED_R2_TO_R3: track 0.00 -> 194.5 mm, vias 0 -> 1
- net LED_R1_TO_R2: track 0.00 -> 194.5 mm
- net LED_DIN: track 0.00 -> 161.9 mm, vias 0 -> 2
- net S_D1: track 0.00 -> 101.9 mm, vias 0 -> 1
- net N_D1: track 0.00 -> 101.8 mm, vias 0 -> 2
- net N_D0: track 0.00 -> 101.6 mm, vias 0 -> 1
- net S_D0: track 0.00 -> 101.2 mm, vias 0 -> 1
- net E_D0: track 0.00 -> 99.5 mm, vias 0 -> 1
- net E_D1: track 0.00 -> 97.3 mm
- net +3V3: track 0.00 -> 57.7 mm
- net ATTINY_TX: track 0.00 -> 54.6 mm
- net ESP_TX: track 0.00 -> 48.9 mm
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- added copper zone on F.Cu, net GND
- removed copper zone on F.Cu, net +5V_LOCAL
